Commit message: got simpler script with no RL stuff for robot reaching to mesh.

File: assistive_gym/envs/assets/bed_mesh/bed_mesh.urdf (robot description, URDF)
Before this commit: robot bed, 2 links, 1 joints
Links:
- added link leg1, mass 0; visual mesh filename=cube.obj scale=0.03 0.03 0.2
- added link leg2, mass 0; visual mesh filename=cube.obj scale=0.03 0.03 0.2
- added link leg3, mass 0; visual mesh filename=cube.obj scale=0.03 0.03 0.2
- added link leg4, mass 0; visual mesh filename=cube.obj scale=0.03 0.03 0.2
Joints:
- added joint mattress_leg1_link: type fixed, parent mattress, child leg1, origin xyz=0.031 0.036 -0.15 rpy=0 0 0, axis 0 0 1, limit lower=0 upper=2 effort=2000 velocity=1
- added joint mattress_leg2_link: type fixed, parent mattress, child leg2, origin xyz=0.031 1.7272 -0.15 rpy=0 0 0, axis 0 0 1, limit lower=0 upper=2 effort=2000 velocity=1
- added joint mattress_leg3_link: type fixed, parent mattress, child leg3, origin xyz=0.8382 0.036 -0.15 rpy=0 0 0, axis 0 0 1, limit lower=0 upper=2 effort=2000 velocity=1
- added joint mattress_leg4_link: type fixed, parent mattress, child leg4, origin xyz=0.8382 1.7272 -0.15 rpy=0 0 0, axis 0 0 1, limit lower=0 upper=2 effort=2000 velocity=1
