Commit message: started to clean up code in human mesh reaching

File: assistive_gym/envs/assets/human_mesh/human_mesh.urdf (robot description, URDF)
Before this commit: robot human, 1 links, 0 joints
Links:
- link human: geometry collision mesh filename=human_vhacd.obj scale=1.0 1.0 1.0; visual mesh filename=human_vhacd.obj scale=1.0 1.0 1.0
